File: the_screamer/screamer.kicad_pcb (KiCad board)
At the start: 4 copper layers, 18 x 14 mm, 15 parts, among them J1 Conn_01x02_Pin, U1 TC2185-3.3VxCTTR, U2 MAX2623EUA+T

Commit message: Add Screamer passive component part numbers
Parts:
- J1: value Conn_01x02_Pin -> 2PH1-02-UA
Changed lines of the file:
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@@
 			)
 		)
-		(property "DKPN" "CONN"
+		(property "DKPN" "A100080CT-ND"
 			(at 0 0 180)
 			(unlocked yes)
@@
 			)
 		)
+		(property "DKPN" "732-7754-1-ND"
+			(at 0 0 180)
+			(unlocked yes)
+			(layer "F.Fab")
+			(hide yes)
+			(effects
+				(font
+					(size 1 1)
+					(thickness 0.15)
+				)
+			)
+		)
 		(property ki_fp_filters "C_*")
 		(sheetname "Root")
@@
 		(sheetname "Root")
 		(sheetfile "screamer.kicad_sch")
-		(attr exclude_from_pos_files)
+		(attr exclude_from_pos_files exclude_from_bom)
 		(fp_circle
 			(center 0 0)
@@
 			)
 		)
+		(property "DKPN" "732-7754-1-ND"
+			(at 0 0 180)
+			(unlocked yes)
+			(layer "F.Fab")
+			(hide yes)
+			(effects
+				(font
+					(size 1 1)
+					(thickness 0.15)
+				)
+			)
+		)
 		(property ki_fp_filters "C_*")
 		(sheetname "Root")
@@
 			)
 		)
+		(property "DKPN" "RMCF0603FT750RCT-ND"
+			(at 0 0 0)
+			(unlocked yes)
+			(layer "F.Fab")
+			(hide yes)
+			(effects
+				(font
+					(size 1 1)
+					(thickness 0.15)
+				)
+			)
+		)
 		(property ki_fp_filters "R_*")
 		(sheetname "Root")
@@
 			)
 		)
-		(property "DKPN" "311-1446-1-ND"
+		(property "DKPN" "732-885012106030CT-ND"
 			(at 0 0 0)
 			(unlocked yes)
@@
 		(sheetname "Root")
 		(sheetfile "screamer.kicad_sch")
-		(attr exclude_from_pos_files)
+		(attr exclude_from_pos_files exclude_from_bom)
 		(fp_circle
 			(center 0 0)
@@
 			)
 		)
-		(property "DKPN" "490-4781-1-ND"
+		(property "DKPN" "732-7983-1-ND"
 			(at 0 0 0)
 			(unlocked yes)
@@
 				(font
 					(size 1.27 1.27)
+				)
+			)
+		)
+		(property "DKPN" "RMCF0603FT1K20CT-ND"
+			(at 0 0 0)
+			(unlocked yes)
+			(layer "F.Fab")
+			(hide yes)
+			(effects
+				(font
+					(size 1 1)
+					(thickness 0.15)
 				)
 			)
@@
 			)
 		)
-		(property "DKPN" "311-1446-1-ND"
+		(property "DKPN" "732-885012106030CT-ND"
 			(at 0 0 180)
 			(unlocked yes)
@@
 			)
 		)
+		(property "DKPN" "175-MAX2623EUA+TCT-ND"
+			(at 0 0 90)
+			(unlocked yes)
+			(layer "B.Fab")
+			(hide yes)
+			(effects
+				(font
+					(size 1 1)
+					(thickness 0.15)
+				)
+				(justify mirror)
+			)
+		)
 		(property ki_fp_filters "21-0036K_MXM 21-0036K_MXM-M 21-0036K_MXM-L")
 		(sheetname "Root")
@@
 			)
 		)
-		(property "Value" "Conn_01x02_Pin"
+		(property "Value" "2PH1-02-UA"
 			(at 0 2.5 -90)
 			(layer "B.Fab")
@@
 			)
 		)
-		(property "DKPN" "STOCK"
+		(property "DKPN" "A100080CT-ND"
 			(at 0 0 90)
 			(unlocked yes)

Commit message: Generated Screamer and Timer BOMs
Both Screamer and Timer have been bumped to V0.1.
Other:
- board text added: "V0.1.0"
- board text removed: "V0.0.3"
Changed lines of the file:
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@@
 	)
 	(paper "A4")
+	(title_block
+		(title "Screamer")
+		(date "2024-05-15")
+		(rev "V0.1.0")
+		(company "Mines Rocket Club")
+		(comment 1 "Andrew Wu")
+	)
 	(layers
 		(0 "F.Cu" signal)
@@
 		(layer "Edge.Cuts")
 	)
-	(gr_text "V0.0.3"
+	(gr_text "V0.1.0"
 		(at 150.5 95 270)
 		(layer "B.SilkS")

Commit message: Fixed custom symbol file paths
In addition to fixing all the file paths I also updated some symbols on the Timer and Screamer, updated the board characteristic tables, added missing 3D models to some components, and did a bit of other file stuff.
Parts:
- moved BT1 7.57 mm to (159.0, 100.0)
Connections:
- net Net-(BT1-+) renamed /BT-
- net Net-(BT1--) renamed /BT+

Commit message: Added automatic revision label to PCBs
Other:
- board text added: "${REVISION}"
- board text removed: "V0.1.0"
Changed lines of the file:
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@@
 		(layer "Edge.Cuts")
 	)
-	(gr_text "V0.1.0"
+	(gr_text "${REVISION}"
 		(at 150.5 95 270)
 		(layer "B.SilkS")
