File: the_guesser/the_guesser.kicad_pcb (KiCad board)
At the start: 2 copper layers, 0 parts

Commit message: Started on Guesser transmitter schematic
Parts:
- added C1: 1u, Capacitor_SMD:C_0603_1608Metric, B.Cu at (249.5, 63.5)
- added C101: 15p, Capacitor_SMD:C_0603_1608Metric, B.Cu at (245.5, 78.5)
- added C111: 100n, Capacitor_SMD:C_0603_1608Metric, B.Cu at (245.5, 81.0)
- added C121: 1p, Capacitor_SMD:C_0603_1608Metric, B.Cu at (245.5, 83.6)
- added C122: 1.5p, Capacitor_SMD:C_0603_1608Metric, B.Cu at (245.5, 86.1)
- added C123: 47p, Capacitor_SMD:C_0603_1608Metric, B.Cu at (241.5, 63.5)
- added C124: 100p, Capacitor_SMD:C_0603_1608Metric, B.Cu at (241.5, 66.0)
- added C125: 0.8p, Capacitor_SMD:C_0603_1608Metric, B.Cu at (260.5, 78.0)
- added C131: 1.5p, Capacitor_SMD:C_0603_1608Metric, B.Cu at (241.5, 71.0)
- added C132: 15p, Capacitor_SMD:C_0603_1608Metric, B.Cu at (210.5, 66.0)
- added C141: 100n, Capacitor_SMD:C_0603_1608Metric, B.Cu at (255.0, 103.8)
- added C151: 100n, Capacitor_SMD:C_0603_1608Metric, B.Cu at (259.0, 107.5)
- added C161: 27p, Capacitor_SMD:C_0603_1608Metric, B.Cu at (208.2, 62.2)
- added C181: 100n, Capacitor_SMD:C_0603_1608Metric, B.Cu at (259.0, 112.0)
- added C2: 10u, Capacitor_SMD:C_0603_1608Metric, B.Cu at (259.0, 81.5)
- added C21: 47p, Capacitor_SMD:C_0603_1608Metric, B.Cu at (213.5, 58.5)
- added C22: 12p, Capacitor_SMD:C_0603_1608Metric, B.Cu at (215.8, 59.2)
- added C24: 3.3p, Capacitor_SMD:C_0603_1608Metric, B.Cu at (215.0, 55.5)
- added C25: 7.5p, Capacitor_SMD:C_0603_1608Metric, B.Cu at (212.0, 57.0)
- added C26: 47p, Capacitor_SMD:C_0603_1608Metric, B.Cu at (209.8, 59.2)
- added C27: 1n, Capacitor_SMD:C_0603_1608Metric, B.Cu at (211.2, 59.2)
- added C28: ???, Capacitor_SMD:C_0603_1608Metric, B.Cu at (209.0, 57.0)
- added C3: 220p, Capacitor_SMD:C_0603_1608Metric, B.Cu at (259.0, 86.0)
- added C30: 1u, Capacitor_SMD:C_0603_1608Metric, B.Cu at (208.2, 59.2)
- added C41: 100n, Capacitor_SMD:C_0603_1608Metric, B.Cu at (245.5, 66.0)
- added C51: 100n, Capacitor_SMD:C_0603_1608Metric, B.Cu at (245.5, 68.5)
- added C52: 12p, Capacitor_SMD:C_0603_1608Metric, B.Cu at (217.2, 59.2)
- added C81: 12p, Capacitor_SMD:C_0603_1608Metric, B.Cu at (245.5, 73.5)
- added C91: 100n, Capacitor_SMD:C_0603_1608Metric, B.Cu at (245.5, 76.0)
- added H1: MountingHole, MountingHole:MountingHole_3.2mm_M3, F.Cu at (202.5, 97.5)
- added H2: MountingHole, MountingHole:MountingHole_3.2mm_M3, F.Cu at (221.5, 97.5)
- added H3: MountingHole, MountingHole:MountingHole_3.2mm_M3, F.Cu at (202.5, 40.5)
- added H4: MountingHole, MountingHole:MountingHole_3.2mm_M3, F.Cu at (221.5, 40.5)
- added J1: USB_B_Mini, Connector_USB:USB_Mini-B_Wuerth_65100516121_Horizontal, F.Cu at (218.0, 50.0)
- added J2: Conn_Coaxial, Connector_Coaxial:SMA_Amphenol_901-143_Horizontal, F.Cu at (204.5, 47.8)
- added J3: RFShield_TwoPieces, RF_Shielding:Laird_Technologies_BMI-S-209-F_29.36x18.50mm, B.Cu at (210.0, 68.0)
- added L1: 1k, Inductor_SMD:L_0603_1608Metric, B.Cu at (241.5, 86.1)
- added L121: 12n, Inductor_SMD:L_0603_1608Metric, B.Cu at (252.0, 103.8)
- added L122: 18n, Inductor_SMD:L_0603_1608Metric, B.Cu at (237.5, 81.0)
- added L130: 1.5n, Inductor_SMD:L_0603_1608Metric, B.Cu at (208.2, 65.2)
- added L131: 12n, Inductor_SMD:L_0603_1608Metric, B.Cu at (253.5, 103.8)
- added L132: 18n, Inductor_SMD:L_0603_1608Metric, B.Cu at (233.5, 63.5)
- added L2: 11n, Inductor_SMD:L_0603_1608Metric, B.Cu at (258.2, 83.8)
- added L21: 22n, Inductor_SMD:L_0603_1608Metric, B.Cu at (213.5, 60.0)
- added L22: 7.5n, Inductor_SMD:L_0603_1608Metric, B.Cu at (215.0, 57.0)
- added L23: 2.9n, Inductor_SMD:L_0603_1608Metric, B.Cu at (212.0, 55.5)
- added L24: 9.1n, Inductor_SMD:L_0603_1608Metric, B.Cu at (209.0, 55.5)
- added L25: 10n, Inductor_SMD:L_0603_1608Metric, B.Cu at (262.8, 77.2)
- added R141: 3.3k, Resistor_SMD:R_0603_1608Metric, B.Cu at (210.5, 64.5)
- added R151: 47, Resistor_SMD:R_0603_1608Metric, B.Cu at (210.5, 63.0)
- added R161: 10, Resistor_SMD:R_0603_1608Metric, B.Cu at (210.5, 61.5)
- added R171: 56k, Resistor_SMD:R_0603_1608Metric, B.Cu at (259.0, 110.5)
- added U2: ESP32-S3, Package_DFN_QFN:QFN-56-1EP_7x7mm_P0.4mm_EP4x4mm, F.Cu at (164.2, 137.2)
- added U3: W25Q128JVS, Package_SO:SOIC-8_5.23x5.23mm_P1.27mm, F.Cu at (174.0, 136.0)
- added U5: CC1101RGPR, locals_but_working_PLEASE:QFN50P400X400X100-21N, B.Cu at (252.0, 110.0)
- added U6: CC1190RGVR, locals_but_working_PLEASE:QFN65P400X400X100-17N, B.Cu at (215.0, 63.8)
- added U7: B39921B3728U410, Filter:Filter_SAW-6_3.8x3.8mm, B.Cu at (267.5, 80.2)
- added X1: STDCRG2-27M, Crystal:Crystal_SMD_3225-4Pin_3.2x2.5mm, B.Cu at (233.5, 92.5)
- added X2: ECS-3953M-400-AU-TR, Crystal:Crystal_SMD_5032-4Pin_5.0x3.2mm, F.Cu at (162.9, 144.3)
Routing:
- net GND: track 0.00 -> 20.2 mm
- net VCC_{CC1190}: track 0.00 -> 10.4 mm
- net VCC_LNA: track 0.00 -> 6.06 mm
- net Net-(C21-Pad1): track 0.00 -> 5.06 mm
- net TR_SW: track 0.00 -> 4.13 mm
- net LNA_IN: track 0.00 -> 3.69 mm
- net Net-(C25-Pad2): track 0.00 -> 3.61 mm
- net PA_OUT: track 0.00 -> 3.56 mm
- net VCC_PA1: track 0.00 -> 2.39 mm
- net VCC_PA2: track 0.00 -> 1.99 mm
- net Net-(U6-BIAS): track 0.00 -> 1.99 mm
- net Net-(J2-In): track 0.00 -> 1.51 mm
- net Net-(C22-Pad1): track 0.00 -> 1.49 mm
- added copper zone on B.Cu, net GND
- added copper zone on F.Cu, net GND
- added copper zone on In1.Cu, net VCC
Other:
- board outline added: 24 x 72 mm
- copper layers 2 -> 4
- board text added: "0"
- board text added: "0 mm"
- board text added: "0.0000 mm / 0.0000 mm"
- board text added: "0.01 mm"
- board text added: "0.02"
- board text added: "0.035 mm"
- board text added: "0.1 mm"
- board text added: "0.3000 mm"
- board text added: "1"
- board text added: "1.24 mm"
- board text added: "1.6000 mm"
- board text added: "156.1423 mm x 73.8183 mm"
- board text added: "3.3"
- board text added: "4"
- board text added: "4.5"
- board text added: "B.Cu"
- board text added: "B.Mask"
- board text added: "B.Paste"
- board text added: "B.Silkscreen"
- board text added: "BOARD CHARACTERISTICS"
- board text added: "Board Thickness:"
- board text added: "Board overall dimensions:"
- board text added: "Bottom Silk Screen"
- board text added: "Bottom Solder Mask"
- board text added: "Bottom Solder Paste"
- board text added: "Castellated pads:"
- board text added: "Color"
- board text added: "Copper Finish:"
- board text added: "Copper Layer Count:"
- board text added: "Dielectric 1"
- board text added: "Dielectric 2"
- board text added: "Dielectric 3"
- board text added: "Edge card connectors:"
- board text added: "Epsilon R"
- board text added: "F.Cu"
- board text added: "F.Mask"
- board text added: "F.Paste"
- board text added: "F.Silkscreen"
- board text added: "FR4"
- board text added: "Impedance Control:"
- board text added: "In1.Cu"
- board text added: "In2.Cu"
- board text added: "Layer Name"
- board text added: "Loss Tangent"
- board text added: "Material"
- board text added: "Min hole diameter:"
- board text added: "Min track/spacing:"
- board text added: "No"
- board text added: "None"
- board text added: "Not specified"
- board text added: "Plated Board Edge:"
- board text added: "Red"
- board text added: "Thickness (mm)"
- board text added: "Top Silk Screen"
- board text added: "Top Solder Mask"
- board text added: "Top Solder Paste"
- board text added: "Type"
- board text added: "copper"
- board text added: "core"
- board text added: "prepreg"
