File: the_pointer/Pointer_Sensors.kicad_sch (KiCad schematic)
At the start: 15 parts, among them J6 BMI-S-209-F, U11 SAM-M8Q, U6 MS5607-02BA, U7 H3LIS200DLTR, U8 BMI088, U9 MMC5883MA

Commit message: Routed Pointer RF transmitter
Parts:
- removed C10, C8: 10u, Capacitor_SMD:C_0603_1608Metric, symbol Device:C_Small
- removed C11, C12: 100n, Capacitor_SMD:C_0603_1608Metric, symbol Device:C_Small
- removed C6, C7: 0.1u, Capacitor_SMD:C_0603_1608Metric, symbol Device:C_Small
- removed C9: 1u, Capacitor_SMD:C_0603_1608Metric, symbol Device:C_Small
- removed J6: BMI-S-209-F, RF_Shielding:Laird_Technologies_BMI-S-209-F_29.36x18.50mm, symbol Device:RFShield_OnePiece
- removed U6: MS5607-02BA, Package_LGA:LGA-8_3x5mm_P1.25mm, symbol Sensor_Pressure:MS5607-02BA
- removed U7: H3LIS200DLTR, locals_but_working_PLEASE:H3LIS200DLTR, symbol Custom_Flight_Computer_Symbols:H3LIS200DLTR
- removed U8: BMI088, locals_but_working_PLEASE:BMI088, symbol Custom_Flight_Computer_Symbols:BMI088
- removed U9: MMC5883MA, locals_but_working_PLEASE:MMC5983MA, symbol Custom_Flight_Computer_Symbols:MMC5983MA
Connections:
- no-connect marks 6 -> 0
